File: POWER.kicad_sch (KiCad schematic)
At the start: 0 parts

Commit message: started connecting board
Parts:
- added D?: D, Diode_SMD:D_SOD-323, symbol Device:D
- added D?: GREEN, LED_SMD:LED_0805_2012Metric, symbol Device:LED
- added D?: RED, LED_SMD:LED_0805_2012Metric, symbol Device:LED
- added R? (x2): 1k, Resistor_SMD:R_0805_2012Metric, symbol Device:R_US
- added R?: 10k, Resistor_SMD:R_0805_2012Metric, symbol Device:R_US
- added U?: MCP73831-2-OT, Package_TO_SOT_SMD:SOT-23-5, symbol Battery_Management:MCP73831-2-OT
- added U?: AP2127K-3.3, Package_TO_SOT_SMD:SOT-23-5, symbol Regulator_Linear:AP2127K-3.3
Connections:
- new net: D?.2 (A), U?.1 (STAT)
- new net: R?.1, U?.5 (PROG)
- new net: D?.1 (K), R?.2 (x2)
- new net +3V3: U?.5 (VOUT)
- new net +BATT: D?.2 (A), U?.3 (VBAT)
- new net GND: R?.1, R?.1, R?.2, U?.2 (GND), U?.2 (VSS)
- new net VBUS: D?.1 (K), D?.2 (A), U?.1 (VIN), U?.3 (EN), U?.4 (VDD)
