File: SENSORS.kicad_sch (KiCad schematic)
At the start: 0 parts

Commit message: finished telemetry
Parts:
- added C? (x2): 1u, Capacitor_SMD:C_0402_1005Metric, symbol Device:C
- added C? (x2): 100n, Capacitor_SMD:C_0402_1005Metric, symbol Device:C
- added U?: LSM6DS3, Package_LGA:LGA-14_3x2.5mm_P0.5mm_LayoutBorder3x4y, symbol Sensor_Motion:LSM6DS3
- added U?: LIS2MDL, Package_LGA:LGA-12_2x2mm_P0.5mm, symbol Sensor_Magnetic_LIS2MDL:LIS2MDL
Connections:
- new net +3V3: C?.2, C?.2, C?.2, C?.2, U?.10 (VDDIO), U?.9 (VDD)
- new net GND: C?.1, C?.1, C?.1, C?.1, U?.11 (NC), U?.12 (NC), U?.2 (NC)

Commit message: Finished Snesors
Parts:
- removed C?: 1u, Capacitor_SMD:C_0402_1005Metric, symbol Device:C
- removed C?: 100n, Capacitor_SMD:C_0402_1005Metric, symbol Device:C
- added C? (x3): 100n, Capacitor_SMD:C_0402_1005Metric, symbol Device:C
- added U?: MS5611-01BA, Package_LGA:LGA-8_3x5mm_P1.25mm, symbol Sensor_Pressure:MS5611-01BA
- C?: value 1u -> 100n
Connections:
- net +3V3: now also U?.2 (SDX), U?.3 (SCX), U?.5 (VDDIO), U?.8 (VDD), C?.1, C?.1, C?.1, U?.1 (VDD)
- net GND: now also U?.6 (GND), U?.6 (GND), U?.7 (GND), U?.8 (GND), C?.2, C?.2, C?.2, U?.2 (PS), U?.3 (GND)
- net SNS_SPI_MISO: now reaches U?.1 (SDO/SA0)
- net SNS_SPI_MISO: now also U?.7 (INT/DRDY/SDO), U?.6 (SDO)
- net LSM6_CS: now reaches U?.12 (CS)
- net SNS_SPI_SCK: now reaches U?.13 (SCL)
- net SNS_SPI_SCK: now also U?.1 (SCL/SPC), U?.8 (SCLK)
- net SNS_SPI_MOSI: now reaches U?.14 (SDA)
- net SNS_SPI_MOSI: now also U?.4 (SDA/SDI/SDO), U?.7 (SDI/SDA)
- net LSM6_INT1: now reaches U?.4 (INT1)
- net LSM6_INT2: now reaches U?.9 (INT2)
- net LIS2_CS: now reaches U?.3 (CS)
- new net MS5611_CS: U?.4 (CSB), U?.5 (CSB)
Other:
- note added: "LIS2MDL"
- note added: "LSM6DSO"
- note added: "MS5611"
- moved on the sheet: C?, U?

Commit message: finished routing
Parts:
- gave numbers to parts that had none: 8
Changed lines of the file:
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@@
   (symbol (lib_id "power:GND") (at 161.29 92.71 0) (unit 1)
     (in_bom yes) (on_board yes) (fields_autoplaced)
-    (property "Reference" "#PWR?" (id 0) (at 161.29 99.06 0)
+    (property "Reference" "#PWR0313" (id 0) (at 161.29 99.06 0)
       (effects (font (size 1.27 1.27)) hide)
     )
@@
   (symbol (lib_id "power:+3V3") (at 161.29 29.21 0) (unit 1)
     (in_bom yes) (on_board yes) (fields_autoplaced)
-    (property "Reference" "#PWR?" (id 0) (at 161.29 33.02 0)
+    (property "Reference" "#PWR0312" (id 0) (at 161.29 33.02 0)
       (effects (font (size 1.27 1.27)) hide)
     )
@@
   (symbol (lib_id "power:+3V3") (at 67.31 129.54 0) (unit 1)
     (in_bom yes) (on_board yes) (fields_autoplaced)
-    (property "Reference" "#PWR?" (id 0) (at 67.31 133.35 0)
+    (property "Reference" "#PWR0305" (id 0) (at 67.31 133.35 0)
       (effects (font (size 1.27 1.27)) hide)
     )
@@
   (symbol (lib_id "Device:C") (at 52.07 139.7 0) (unit 1)
     (in_bom yes) (on_board yes) (fields_autoplaced)
-    (property "Reference" "C?" (id 0) (at 55.88 138.4299 0)
+    (property "Reference" "C301" (id 0) (at 55.88 138.4299 0)
       (effects (font (size 1.27 1.27)) (justify left))
     )
@@
   (symbol (lib_id "power:+3V3") (at 34.29 55.88 0) (unit 1)
     (in_bom yes) (on_board yes) (fields_autoplaced)
-    (property "Reference" "#PWR?" (id 0) (at 34.29 59.69 0)
+    (property "Reference" "#PWR0301" (id 0) (at 34.29 59.69 0)
       (effects (font (size 1.27 1.27)) hide)
     )
@@
   (symbol (lib_id "Sensor_Pressure:MS5611-01BA") (at 67.31 149.86 0) (unit 1)
     (in_bom yes) (on_board yes) (fields_autoplaced)
-    (property "Reference" "U?" (id 0) (at 76.2 148.5899 0)
+    (property "Reference" "U301" (id 0) (at 76.2 148.5899 0)
       (effects (font (size 1.27 1.27)) (justify left))
     )
@@
   (symbol (lib_id "power:GND") (at 80.01 52.07 0) (unit 1)
     (in_bom yes) (on_board yes) (fields_autoplaced)
-    (property "Reference" "#PWR?" (id 0) (at 80.01 58.42 0)
+    (property "Reference" "#PWR0309" (id 0) (at 80.01 58.42 0)
       (effects (font (size 1.27 1.27)) hide)
     )
@@
   (symbol (lib_id "power:GND") (at 62.23 52.07 0) (unit 1)
     (in_bom yes) (on_board yes) (fields_autoplaced)
-    (property "Reference" "#PWR?" (id 0) (at 62.23 58.42 0)
+    (property "Reference" "#PWR0303" (id 0) (at 62.23 58.42 0)
       (effects (font (size 1.27 1.27)) hide)
     )
@@
   (symbol (lib_id "power:GND") (at 139.7 46.99 0) (unit 1)
     (in_bom yes) (on_board yes) (fields_autoplaced)
-    (property "Reference" "#PWR?" (id 0) (at 139.7 53.34 0)
+    (property "Reference" "#PWR0310" (id 0) (at 139.7 53.34 0)
       (effects (font (size 1.27 1.27)) hide)
     )
@@
   (symbol (lib_id "power:GND") (at 171.45 44.45 0) (unit 1)
     (in_bom yes) (on_board yes) (fields_autoplaced)
-    (property "Reference" "#PWR?" (id 0) (at 171.45 50.8 0)
+    (property "Reference" "#PWR0314" (id 0) (at 171.45 50.8 0)
       (effects (font (size 1.27 1.27)) hide)
     )
@@
   (symbol (lib_id "Sensor_Motion:LSM6DS3") (at 69.85 69.85 0) (unit 1)
     (in_bom yes) (on_board yes) (fields_autoplaced)
-    (property "Reference" "U?" (id 0) (at 87.63 55.6512 0))
+    (property "Reference" "U302" (id 0) (at 87.63 55.6512 0))
     (property "Value" "LSM6DS3" (id 1) (at 87.63 58.1912 0))
     (property "Footprint" "Package_LGA:LGA-14_3x2.5mm_P0.5mm_LayoutBorder3x4y" (id 2) (at 59.69 87.63 0)
@@
   (symbol (lib_id "power:+3V3") (at 67.31 39.37 0) (unit 1)
     (in_bom yes) (on_board yes) (fields_autoplaced)
-    (property "Reference" "#PWR?" (id 0) (at 67.31 43.18 0)
+    (property "Reference" "#PWR0304" (id 0) (at 67.31 43.18 0)
       (effects (font (size 1.27 1.27)) hide)
     )
@@
   (symbol (lib_id "power:+3V3") (at 74.93 39.37 0) (unit 1)
     (in_bom yes) (on_board yes) (fields_autoplaced)
-    (property "Reference" "#PWR?" (id 0) (at 74.93 43.18 0)
+    (property "Reference" "#PWR0308" (id 0) (at 74.93 43.18 0)
       (effects (font (size 1.27 1.27)) hide)
     )
@@
   (symbol (lib_id "power:GND") (at 196.85 90.17 0) (unit 1)
     (in_bom yes) (on_board yes) (fields_autoplaced)
-    (property "Reference" "#PWR?" (id 0) (at 196.85 96.52 0)
+    (property "Reference" "#PWR0315" (id 0) (at 196.85 96.52 0)
       (effects (font (size 1.27 1.27)) hide)
     )
@@
   (symbol (lib_id "Device:C") (at 62.23 45.72 0) (unit 1)
     (in_bom yes) (on_board yes) (fields_autoplaced)
-    (property "Reference" "C?" (id 0) (at 66.04 44.4499 0)
+    (property "Reference" "C302" (id 0) (at 66.04 44.4499 0)
       (effects (font (size 1.27 1.27)) (justify left))
     )
@@
   (symbol (lib_id "power:GND") (at 69.85 90.17 0) (unit 1)
     (in_bom yes) (on_board yes) (fields_autoplaced)
-    (property "Reference" "#PWR?" (id 0) (at 69.85 96.52 0)
+    (property "Reference" "#PWR0307" (id 0) (at 69.85 96.52 0)
       (effects (font (size 1.27 1.27)) hide)
     )
@@
   (symbol (lib_id "power:GND") (at 39.37 154.94 0) (unit 1)
     (in_bom yes) (on_board yes) (fields_autoplaced)
-    (property "Reference" "#PWR?" (id 0) (at 39.37 161.29 0)
+    (property "Reference" "#PWR0302" (id 0) (at 39.37 161.29 0)
       (effects (font (size 1.27 1.27)) hide)
     )
@@
   (symbol (lib_id "Device:C") (at 171.45 38.1 180) (unit 1)
     (in_bom yes) (on_board yes) (fields_autoplaced)
-    (property "Reference" "C?" (id 0) (at 175.26 36.8299 0)
+    (property "Reference" "C305" (id 0) (at 175.26 36.8299 0)
       (effects (font (size 1.27 1.27)) (justify right))
     )
@@
   (symbol (lib_id "Sensor_Magnetic_LIS2MDL:LIS2MDL") (at 166.37 72.39 0) (unit 1)
     (in_bom yes) (on_board yes) (fields_autoplaced)
-    (property "Reference" "U?" (id 0) (at 160.7694 54.61 0)
+    (property "Reference" "U303" (id 0) (at 160.7694 54.61 0)
       (effects (font (size 1.27 1.27)) (justify left))
     )
@@
   (symbol (lib_id "Device:C") (at 139.7 38.1 180) (unit 1)
     (in_bom yes) (on_board yes) (fields_autoplaced)
-    (property "Reference" "C?" (id 0) (at 143.51 36.8299 0)
+    (property "Reference" "C304" (id 0) (at 143.51 36.8299 0)
       (effects (font (size 1.27 1.27)) (justify right))
     )
@@
   (symbol (lib_id "Device:C") (at 80.01 45.72 0) (unit 1)
     (in_bom yes) (on_board yes) (fields_autoplaced)
-    (property "Reference" "C?" (id 0) (at 83.82 44.4499 0)
+    (property "Reference" "C303" (id 0) (at 83.82 44.4499 0)
       (effects (font (size 1.27 1.27)) (justify left))
     )
@@
   (symbol (lib_id "power:GND") (at 67.31 165.1 0) (unit 1)
     (in_bom yes) (on_board yes) (fields_autoplaced)
-    (property "Reference" "#PWR?" (id 0) (at 67.31 171.45 0)
+    (property "Reference" "#PWR0306" (id 0) (at 67.31 171.45 0)
       (effects (font (size 1.27 1.27)) hide)
     )
@@
   (symbol (lib_id "power:+3V3") (at 153.67 29.21 0) (unit 1)
     (in_bom yes) (on_board yes) (fields_autoplaced)
-    (property "Reference" "#PWR?" (id 0) (at 153.67 33.02 0)
-      (effects (font (size 1.27 1.27)) hide)
-    )
+    (property "Reference" "#PWR0311" (id 0) (at 153.67 33.02 0)
+      (effects (font (size 1.27 1.27)) hide)
+    )
