File: TELEMETRY.kicad_sch (KiCad schematic)
At the start: 7 parts

Commit message: finished routing
Parts:
- U401: renamed from U?; footprint (none) -> RF_Module:HOPERF_RFM9XW_SMD
- gave numbers to parts that had none: 6
Connections:
- net GPS_SAFEBOOT: no longer U402.19 (EXTINT)
- new net GPS_EXTINT: U402.19 (EXTINT)
Changed lines of the file:
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@@
     (effects (font (size 1.27 1.27)) (justify left))
   )
-  (hierarchical_label "GPS_SAFEBOOT" (shape input) (at 170.18 95.25 180)
+  (hierarchical_label "GPS_EXTINT" (shape input) (at 170.18 95.25 180)
     (effects (font (size 1.27 1.27)) (justify right))
   )
@@
   (symbol (lib_id "Device:C") (at 43.18 78.74 180) (unit 1)
     (in_bom yes) (on_board yes) (fields_autoplaced)
-    (property "Reference" "C?" (id 0) (at 46.99 77.4699 0)
+    (property "Reference" "C401" (id 0) (at 46.99 77.4699 0)
       (effects (font (size 1.27 1.27)) (justify right))
     )
@@
   (symbol (lib_id "power:+3V3") (at 180.34 64.77 0) (unit 1)
     (in_bom yes) (on_board yes) (fields_autoplaced)
-    (property "Reference" "#PWR?" (id 0) (at 180.34 68.58 0)
+    (property "Reference" "#PWR0405" (id 0) (at 180.34 68.58 0)
       (effects (font (size 1.27 1.27)) hide)
     )
@@
   (symbol (lib_id "Device:C") (at 172.72 77.47 0) (unit 1)
     (in_bom yes) (on_board yes) (fields_autoplaced)
-    (property "Reference" "C?" (id 0) (at 176.53 76.1999 0)
+    (property "Reference" "C403" (id 0) (at 176.53 76.1999 0)
       (effects (font (size 1.27 1.27)) (justify left))
     )
@@
   (symbol (lib_id "power:GND") (at 119.38 97.79 0) (unit 1)
     (in_bom yes) (on_board yes) (fields_autoplaced)
-    (property "Reference" "#PWR?" (id 0) (at 119.38 104.14 0)
+    (property "Reference" "#PWR0403" (id 0) (at 119.38 104.14 0)
       (effects (font (size 1.27 1.27)) hide)
     )
@@
   (symbol (lib_id "power:GND") (at 168.91 86.36 0) (unit 1)
     (in_bom yes) (on_board yes) (fields_autoplaced)
-    (property "Reference" "#PWR?" (id 0) (at 168.91 92.71 0)
+    (property "Reference" "#PWR0404" (id 0) (at 168.91 92.71 0)
       (effects (font (size 1.27 1.27)) hide)
     )
@@
   (symbol (lib_id "power:+3V3") (at 80.01 59.69 0) (unit 1)
     (in_bom yes) (on_board yes) (fields_autoplaced)
-    (property "Reference" "#PWR?" (id 0) (at 80.01 63.5 0)
+    (property "Reference" "#PWR0401" (id 0) (at 80.01 63.5 0)
       (effects (font (size 1.27 1.27)) hide)
     )
@@
   (symbol (lib_id "power:GND") (at 204.47 82.55 0) (unit 1)
     (in_bom yes) (on_board yes) (fields_autoplaced)
-    (property "Reference" "#PWR?" (id 0) (at 204.47 88.9 0)
+    (property "Reference" "#PWR0408" (id 0) (at 204.47 88.9 0)
       (effects (font (size 1.27 1.27)) hide)
     )
@@
   (symbol (lib_id "Device:C") (at 204.47 77.47 0) (unit 1)
     (in_bom yes) (on_board yes)
-    (property "Reference" "C?" (id 0) (at 198.12 76.2 0)
+    (property "Reference" "C404" (id 0) (at 198.12 76.2 0)
       (effects (font (size 1.27 1.27)) (justify left))
     )
@@
   (symbol (lib_id "power:GND") (at 185.42 116.84 0) (unit 1)
     (in_bom yes) (on_board yes) (fields_autoplaced)
-    (property "Reference" "#PWR?" (id 0) (at 185.42 123.19 0)
+    (property "Reference" "#PWR0406" (id 0) (at 185.42 123.19 0)
       (effects (font (size 1.27 1.27)) hide)
     )
@@
   (symbol (lib_id "Device:C") (at 165.1 77.47 0) (unit 1)
     (in_bom yes) (on_board yes)
-    (property "Reference" "C?" (id 0) (at 158.75 76.2 0)
+    (property "Reference" "C402" (id 0) (at 158.75 76.2 0)
       (effects (font (size 1.27 1.27)) (justify left))
     )
@@
   (symbol (lib_id "RF_GPS:SAM-M8Q") (at 185.42 97.79 0) (unit 1)
     (in_bom yes) (on_board yes) (fields_autoplaced)
-    (property "Reference" "U?" (id 0) (at 187.4394 110.49 0)
+    (property "Reference" "U402" (id 0) (at 187.4394 110.49 0)
       (effects (font (size 1.27 1.27)) (justify left))
     )
@@
   (symbol (lib_id "power:GND") (at 80.01 101.6 0) (unit 1)
     (in_bom yes) (on_board yes) (fields_autoplaced)
-    (property "Reference" "#PWR?" (id 0) (at 80.01 107.95 0)
+    (property "Reference" "#PWR0402" (id 0) (at 80.01 107.95 0)
       (effects (font (size 1.27 1.27)) hide)
     )
@@
   (symbol (lib_id "RF_Module:RFM96W-433S2") (at 80.01 81.28 0) (unit 1)
     (in_bom yes) (on_board yes) (fields_autoplaced)
-    (property "Reference" "U?" (id 0) (at 82.0294 66.04 0)
+    (property "Reference" "U401" (id 0) (at 82.0294 66.04 0)
       (effects (font (size 1.27 1.27)) (justify left))
     )
@@
       (effects (font (size 1.27 1.27)) (justify left))
     )
-    (property "Footprint" "" (id 2) (at -3.81 39.37 0)
+    (property "Footprint" "RF_Module:HOPERF_RFM9XW_SMD" (id 2) (at -3.81 39.37 0)
       (effects (font (size 1.27 1.27)) hide)
     )
@@
   (symbol (lib_id "Connector:Conn_Coaxial") (at 119.38 73.66 0) (unit 1)
     (in_bom yes) (on_board yes) (fields_autoplaced)
-    (property "Reference" "J?" (id 0) (at 121.92 72.6831 0)
+    (property "Reference" "J401" (id 0) (at 121.92 72.6831 0)
       (effects (font (size 1.27 1.27)) (justify left))
     )
@@
   (symbol (lib_id "power:+3V0") (at 190.5 64.77 0) (unit 1)
     (in_bom yes) (on_board yes) (fields_autoplaced)
-    (property "Reference" "#PWR?" (id 0) (at 190.5 68.58 0)
-      (effects (font (size 1.27 1.27)) hide)
-    )
+    (property "Reference" "#PWR0407" (id 0) (at 190.5 68.58 0)
+      (effects (font (size 1.27 1.27)) hide)
+    )
